File: pcb/synth123.sch (KiCad schematic (older format))
At the start: 29 parts, among them IC1 ATTINY4313-P, IC2 PC817, IC3 MCP4802-E/P, K1 STEREO/MONO, P1 POWER, P2 MIDI_IN, P3 ISP, P4 AUDIO_CONNECTOR, U1 7805, X1 20MHz

Commit message: Updated KiCad files.
Connections:
- net at C9.2: now also P4.2; no longer P4.5
- net at C10.2: now also P4.5; no longer P4.2
Changed lines of the file:
@@
-EESchema Schematic File Version 2  date Sat 11 May 2013 11:21:18 PM CEST
+EESchema Schematic File Version 2  date Sat 18 May 2013 11:54:08 AM CEST
 LIBS:attiny4313-p
 LIBS:power
@@
 Sheet 1 1
 Title "Synth123"
-Date "11 may 2013"
+Date "18 may 2013"
 Rev "0.1"
 Comp "Martin Åberg"
@@
 	5850 4550 4800 4550
 Wire Wire Line
-	9250 4650 9250 4450
-Wire Wire Line
-	9250 4450 8800 4450
-Wire Wire Line
 	9250 5050 9250 5150
 Wire Wire Line
@@
 Connection ~ 7800 1800
 Connection ~ 7400 2700
-Wire Wire Line
-	9250 4950 8800 4950
 Wire Wire Line
 	2600 7050 2600 7350
@@
 Connection ~ 8000 4950
 Connection ~ 4400 6450
+Wire Wire Line
+	8800 4450 9150 4450
+Wire Wire Line
+	9150 4450 9150 4950
+Wire Wire Line
+	9150 4950 9250 4950
+Wire Wire Line
+	8800 4950 9050 4950
+Wire Wire Line
+	9050 4950 9050 4650
+Wire Wire Line
+	9050 4650 9250 4650
 $EndSCHEMATC
